File: kicad/mss-xcade/mss-xcade-interface.kicad_sch (KiCad schematic)
At the start: 117 parts

Commit message: More updates
Parts:
- removed J? (x2): 8P8C, RJ45_Amphenol_54602-x08_Horizontal, symbol Connector:8P8C
- added J? (x2): 8P8C, RJ45_Amphenol_54602-x08_Horizontal, symbol Connector:8P8C
- added JP? (x4): SolderJumper_2_Bridged, symbol Jumper:SolderJumper_2_Bridged
Connections:
- net GND2: now also J?.5, J?.5, JP?.1 (A), JP?.1 (A), JP?.1 (A), JP?.1 (A); no longer J?.7, J?.7
- net at R?.1, R?.1: now also J?.1 (x2)
- net at Q?.3 (D): now also J?.6 (x2)
- net at R?.1, R?.1: now also J?.2 (x2)
- net at Q?.3 (D), R?.1, R?.1: now also J?.4 (x2)
- net at Q?.3 (D), R?.1, R?.1: now also J?.8 (x2)
- net at Q?.3 (D): now also J?.3 (x2)
- new net: J?.7, JP?.2 (B) (x4)
Other:
- moved on the sheet: J?

Commit message: Refactor signal drivers to their own schematic and add picoblade connectors
Parts:
- added R? (x4): 0 ohm, Resistor_SMD:R_0805_2012Metric, symbol Device:R_US
- gave numbers to parts that had none: 105
Connections:
- net +5V: now also R?.2
- net +5VD: now also R?.1
- net GND: now also C14.2, U8.1 (VIN-), U8.2 (VIN-), U8.3 (VIN-), R?.2
- net GND2: now also R?.1; no longer C14.2, U8.1 (VIN-), U8.2 (VIN-), U8.3 (VIN-)
- net SCL: now also R?.2
- net SDA: now also R?.2
- net at R57.1, U12.7 (SDA2): now also U13.23 (SDA), U16.23 (SDA), R?.1; no longer U13.22 (SCL), U16.22 (SCL)
- net at R56.1, U12.6 (SCL2): now also U13.22 (SCL), U16.22 (SCL), R?.1; no longer U13.23 (SDA), U16.23 (SDA)
Other:
- note added: "Note: Install two zero ohm jumpers if isolation not required"

Commit message: First cut of xcade PCB
Parts:
- removed C14: 10uF, Capacitor_SMD:C_0805_2012Metric, symbol Device:C
- removed C23, C24: 0.1uF, Capacitor_SMD:C_0805_2012Metric, symbol Device:C
- removed D12: GREEN LED, LED_SMD:LED_0805_2012Metric, symbol Device:LED
- removed R36, R54, R55, R56, R57: 1k, Resistor_SMD:R_0805_2012Metric, symbol Device:R_US
- removed R? (x4): 0 ohm, Resistor_SMD:R_0805_2012Metric, symbol Device:R_US
- removed U12: ISO1641, Package_SO:SOIC-8_3.9x4.9mm_P1.27mm, symbol Isolator:ISO1541
- removed U8: R05C1TF05S-R, ISE_UltraLibrarian:12L-LGA_RxxC1TFxxS_RCP, symbol ISE_UltraLibrarian:R05C1TF05S-R
- added unit 6 of U10
- added unit 1 of U10
- added unit 1 of U6
- added unit 6 of U6
- added unit 1 of U7
- added unit 6 of U7
- added unit 6 of U9
- added unit 1 of U9
- D9: renamed from D11; footprint Diode_SMD:D_SOD-123 -> ISE_Generic:SOD-123T
- JP1: renamed from JP25; footprint (none) -> Jumper:SolderJumper-2_P1.3mm_Bridged_RoundedPad1.0x1.5mm
- JP2: renamed from JP26; footprint (none) -> Jumper:SolderJumper-2_P1.3mm_Bridged_RoundedPad1.0x1.5mm
- JP3: renamed from JP27; footprint (none) -> Jumper:SolderJumper-2_P1.3mm_Bridged_RoundedPad1.0x1.5mm
- JP4: renamed from JP28; footprint (none) -> Jumper:SolderJumper-2_P1.3mm_Bridged_RoundedPad1.0x1.5mm
- U10: renamed from U15; footprint (none) -> Package_SO:SO-16_3.9x9.9mm_P1.27mm
- U11: renamed from U16; value PCA9555D -> TCA9555PWR; footprint Package_SO:SOIC-24W_7.5x15.4mm_P1.27mm -> Package_SO:TSSOP-24_4.4x7.8mm_P0.65mm
- U6: renamed from U10; footprint (none) -> Package_SO:SO-16_3.9x9.9mm_P1.27mm
- U7: renamed from U11; footprint (none) -> Package_SO:SO-16_3.9x9.9mm_P1.27mm
- U8: renamed from U13; value PCA9555D -> TCA9555PWR; footprint Package_SO:SOIC-24W_7.5x15.4mm_P1.27mm -> Package_SO:TSSOP-24_4.4x7.8mm_P0.65mm
- U9: renamed from U14; footprint (none) -> Package_SO:SO-16_3.9x9.9mm_P1.27mm
- renumbered C15 to C11, C16 to C12, C17 to C13, C18 to C14, C19 to C15, C20 to C16, C21 to C17, C22 to C18, C25 to C19, C26 to C20, C27 to C21, C28 to C22, C29 to C23, C30 to C24, C31 to C25, C32 to C26, C33 to C27, C34 to C28, C35 to C29, C36 to C30, C37 to C31, C38 to C32, C39 to C33, C40 to C34, J32 to J10, J29 to J7, J30 to J8, J31 to J9, Q3 to Q1, Q12 to Q10, Q13 to Q11, Q14 to Q12, Q15 to Q13, Q16 to Q14, Q17 to Q15, Q18 to Q16, Q4 to Q2, Q5 to Q3, Q6 to Q4, Q7 to Q5, Q8 to Q6, Q9 to Q7, Q10 to Q8, Q11 to Q9, R37 to R13, R38 to R14, R39 to R15, R40 to R16, R41 to R17, R42 to R18, R43 to R19, R44 to R20, R45 to R21, R46 to R22, R47 to R23, R48 to R24, R49 to R25, R50 to R26, R51 to R27, R52 to R28, R53 to R29, R58 to R30, R59 to R31, R60 to R32, R61 to R33, R62 to R34, R63 to R35, R64 to R36, R65 to R37, R66 to R38, R67 to R39, R68 to R40, R69 to R41, R70 to R42, R71 to R43, R72 to R44, R73 to R45, R74 to R46, R75 to R47, R76 to R48, R77 to R49, U9 to U5
Connections:
- net +5VD is gone; now on net +5V: C11.1, C19.1, C28.1, C31.1, C32.1, C33.1, C34.1, L2.1, U10.1 (VCC), U11.21 (A0), U11.24 (VDD), U5.4 (~{SHDN}), U5.5 (IN), U6.1 (VCC), U7.1 (VCC), U8.24 (VDD), U9.1 (VCC)
- net GND2 is gone; now on net GND: C11.2, C12.2, C13.2, C14.2, C15.2, C16.2, C17.2, C18.2, C19.2, C20.2, C21.2, C22.2, C23.2, C24.2, C25.2, C26.2, C27.2, C28.2, C29.2, C30.2, J10.5, J7.5, J8.5, J9.5, JP1.1 (A), JP2.1 (A), JP3.1 (A), JP4.1 (A), Q1.2 (S), Q10.2 (S), Q11.2 (S), Q12.2 (S), Q13.2 (S), Q14.2 (S), Q15.2 (S), Q16.2 (S), Q2.2 (S), Q3.2 (S), Q4.2 (S), Q5.2 (S), Q6.2 (S), Q7.2 (S), Q8.2 (S), Q9.2 (S), R27.1, U10.8 (VSS), U11.12 (VSS), U11.2 (A1), U11.3 (A2), U5.2 (GND), U6.8 (VSS), U7.8 (VSS), U8.12 (VSS), U8.2 (A1), U8.21 (A0), U8.3 (A2), U9.8 (VSS)
- net GND: now also U10.14, U10.3, U6.14, U6.3, U7.14, U7.3, U9.14, U9.3
- net MSS1_AA_IN: now also U7.4, U8.4 (IO0_0); no longer U7.2, U8.6 (IO0_2)
- net MSS1_AA_OUT: now also U8.9 (IO0_5); no longer U8.10 (IO0_6)
- net MSS1_A_IN: now also U7.6; no longer U7.4
- net MSS1_A_OUT: now also U8.11 (IO0_7); no longer U8.9 (IO0_5)
- net MSS1_DA_IN: now also U7.12; no longer U7.10
- net MSS1_DA_OUT: now also U8.8 (IO0_4); no longer U8.11 (IO0_7)
- net MSS1_S_IN: now also U7.10, U8.6 (IO0_2); no longer U7.6, U8.4 (IO0_0)
- net MSS1_S_OUT: now also U8.10 (IO0_6); no longer U8.8 (IO0_4)
- net MSS2_AA_IN: now also U6.4, U8.13 (IO1_0); no longer U6.2, U8.15 (IO1_2)
- net MSS2_AA_OUT: now also U8.18 (IO1_5); no longer U8.19 (IO1_6)
- net MSS2_A_IN: now also U6.6; no longer U6.4
- net MSS2_A_OUT: now also U8.20 (IO1_7); no longer U8.18 (IO1_5)
- net MSS2_DA_IN: now also U6.12; no longer U6.10
- net MSS2_DA_OUT: now also U8.17 (IO1_4); no longer U8.20 (IO1_7)
- net MSS2_S_IN: now also U6.10, U8.15 (IO1_2); no longer U6.6, U8.13 (IO1_0)
- net MSS2_S_OUT: now also U8.19 (IO1_6); no longer U8.17 (IO1_4)
- net MSS3_AA_IN: now also U10.4, U11.4 (IO0_0); no longer U10.2, U11.6 (IO0_2)
- net MSS3_AA_OUT: now also U11.9 (IO0_5); no longer U11.10 (IO0_6)
- net MSS3_A_IN: now also U10.6; no longer U10.4
- net MSS3_A_OUT: now also U11.11 (IO0_7); no longer U11.9 (IO0_5)
- net MSS3_DA_IN: now also U10.12; no longer U10.10
- net MSS3_DA_OUT: now also U11.8 (IO0_4); no longer U11.11 (IO0_7)
- net MSS3_S_IN: now also U10.10, U11.6 (IO0_2); no longer U10.6, U11.4 (IO0_0)
- net MSS3_S_OUT: now also U11.10 (IO0_6); no longer U11.8 (IO0_4)
- net MSS4_AA_IN: now also U11.13 (IO1_0), U9.4; no longer U11.15 (IO1_2), U9.2
- net MSS4_AA_OUT: now also U11.18 (IO1_5); no longer U11.19 (IO1_6)
- net MSS4_A_IN: now also U9.6; no longer U9.4
- net MSS4_A_OUT: now also U11.20 (IO1_7); no longer U11.18 (IO1_5)
- net MSS4_DA_IN: now also U9.12; no longer U9.10
- net MSS4_DA_OUT: now also U11.17 (IO1_4); no longer U11.20 (IO1_7)
- net MSS4_S_IN: now also U11.15 (IO1_2), U9.10; no longer U11.13 (IO1_0), U9.6
- net MSS4_S_OUT: now also U11.19 (IO1_6); no longer U11.17 (IO1_4)
- net SCL: now also U11.22 (SCL), U8.22 (SCL)
- net SDA: now also U11.23 (SDA), U8.23 (SDA)
- net at C22.1, R40.2: now also U9.5; no longer U9.3
- net at C24.1, R44.2: now also U9.9; no longer U9.7
- net at C13.1, R23.2: now also U6.5; no longer U6.3
- net at C25.1, R41.2: now also U10.5; no longer U10.3
- net at C21.1, R33.2: now also U7.11; no longer U7.9
- net at C27.1, R45.2: now also U10.9; no longer U10.7
- net at C23.1, R42.2: now also U9.7; no longer U9.5
- net at C14.1, R25.2: now also U6.7; no longer U6.5
- net at C16.1, R24.2: now also U7.5; no longer U7.3
- net at C20.1, R32.2: now also U6.11; no longer U6.9
- net at C30.1, R49.2: now also U10.11; no longer U10.9
- net at C26.1, R43.2: now also U10.7; no longer U10.5
- net at C15.1, R28.2: now also U6.9; no longer U6.7
- net at C17.1, R26.2: now also U7.7; no longer U7.5
- net at C18.1, R29.2: now also U7.9; no longer U7.7
- net at C29.1, R48.2: now also U9.11; no longer U9.9
Other:
- note removed: "Note: Install two zero ohm jumpers if isolation not required"
