File: kicad/mss-xcade/mss-xcade-signal-drivers.kicad_sch (KiCad schematic)
At the start: 92 parts

Commit message: First cut of xcade PCB
Parts:
- removed C?: 1uF, Capacitor_SMD:C_0805_2012Metric, symbol Device:C
- removed D? (x2): AMBER, LED_SMD:LED_0805_2012Metric, symbol Device:LED
- removed J? (x2): Screw_Terminal_01x02, TerminalBlock_MetzConnect:TerminalBlock_MetzConnect_Type059_RT06303HBWC_1x03_P3.50mm_Horizontal, symbol Connector:Screw_Terminal_01x03
- removed J?: Screw_Terminal_01x08, symbol Connector:Screw_Terminal_01x08
- removed R? (x2): 1k, Resistor_SMD:R_0805_2012Metric, symbol Device:R_US
- removed U? (x2): PCA9635, Package_SO:TSSOP-28_4.4x9.7mm_P0.65mm, symbol Driver_LED:PCA9635
- added J31: AVR-ISP, Connector:Tag-Connect_TC2030-IDC-NL_2x03_P1.27mm_Vertical, symbol ISE_Generic:Conn_AVR_TagConnect_TC2030
- added J42: Screw_Terminal_01x08, TerminalBlock_TE-Connectivity:TerminalBlock_TE_282834-8_1x08_P2.54mm_Horizontal, symbol Connector:Screw_Terminal_01x08
- added R75: 10k, Resistor_SMD:R_0805_2012Metric, symbol Device:R_US
- added U12: ATtiny88-A, Package_QFP:TQFP-32_7x7mm_P0.8mm, symbol MCU_Microchip_ATtiny:ATtiny88-A
- U13: renamed from U?; value PCA9555D -> TCA9555PWR; footprint Package_SO:SOIC-24W_7.5x15.4mm_P1.27mm -> Package_SO:TSSOP-24_4.4x7.8mm_P0.65mm
- gave numbers to parts that had none: 81
Connections:
- net +5V: now also J32.MP (MountPin), J33.2 (Pin_2), J33.MP (MountPin), J34.2 (Pin_2), J34.MP (MountPin), J35.MP (MountPin), J36.MP (MountPin), J37.2 (Pin_2), J37.MP (MountPin), J38.2 (Pin_2), J38.MP (MountPin), J39.MP (MountPin), J40.MP (MountPin), J41.MP (MountPin), J31.2 (VCC), J42.8 (Pin_8), R75.1, U12.18 (AVCC), U12.4 (VCC)
- net A1_SIGNAL_G: now also U12.32 (PD2)
- net A1_SIGNAL_R: now also U12.30 (PD0)
- net A1_SIGNAL_Y: now also U12.31 (PD1)
- net A2_SIGNAL_G: now also U12.3 (PA2)
- net A2_SIGNAL_R: now also U12.1 (PD3)
- net A2_SIGNAL_Y: now also U12.2 (PD4)
- net B1_SIGNAL_G: now also U12.8 (PB7)
- net B1_SIGNAL_R: now also U12.6 (PA3)
- net B1_SIGNAL_Y: now also U12.7 (PB6)
- net B2_SIGNAL_G: now also U12.11 (PD7)
- net B2_SIGNAL_R: now also U12.9 (PD5)
- net B2_SIGNAL_Y: now also U12.10 (PD6)
- net C1_SIGNAL_G: now also U12.14 (PB2)
- net C1_SIGNAL_R: now also U12.12 (PB0)
- net C1_SIGNAL_Y: now also U12.13 (PB1)
- net C2_SIGNAL_G: now also J31.3 (SCK), U12.17 (PB5)
- net C2_SIGNAL_R: now also J31.4 (MOSI), U12.15 (PB3)
- net C2_SIGNAL_Y: now also J31.1 (MISO), U12.16 (PB4)
- net COM_SENSE: now also U12.19 (PA0); no longer U13.20 (IO1_7)
- net D1_SIGNAL_G: now also U12.23 (PC0)
- net D1_SIGNAL_R: now also U12.20 (PC7)
- net D1_SIGNAL_Y: now also U12.22 (PA1)
- net D2_SIGNAL_G: now also U12.26 (PC3)
- net D2_SIGNAL_R: now also U12.24 (PC1)
- net D2_SIGNAL_Y: now also U12.25 (PC2)
- net GND: now also J31.6 (GND), J42.1 (Pin_1), U12.21 (GND), U12.5 (GND); no longer J32.MP (MountPin), J33.MP (MountPin), J34.MP (MountPin), J35.MP (MountPin), J36.MP (MountPin), J37.MP (MountPin), J38.MP (MountPin), J39.MP (MountPin), J40.MP (MountPin), J41.MP (MountPin)
- net SCL: now also U12.28 (PC5)
- net SDA: now also U12.27 (PC4)
- net SENSOR_IN_10: now also J42.7 (Pin_7)
- net SENSOR_IN_11: now also J42.6 (Pin_6)
- net SENSOR_IN_12: now also J42.5 (Pin_5)
- net SENSOR_IN_13: now also J42.4 (Pin_4)
- net SENSOR_IN_14: now also J42.3 (Pin_3)
- new net: J31.5 (~{RESET}), R75.2, U12.29 (~{RESET}/PC6)
- new net SENSOR_IN_15: J42.2 (Pin_2), U13.20 (IO1_7)
Other:
- note added: "Atlas Signal Connector for Signal A Lower Molex Picoblade 1 - Yellow 2 - Green 3 - Red 4 - Common"
- note added: "Atlas Signal Connector for Signal B Lower Molex Picoblade 1 - Yellow 2 - Green 3 - Red 4 - Common"
- note added: "Atlas Signal Connector for Signal B Upper Molex Picoblade 1 - Yellow 2 - Green 3 - Red 4 - Common"
- note added: "Atlas Signal Connector for Signal C Lower Molex Picoblade 1 - Yellow 2 - Green 3 - Red 4 - Common"
- note added: "Atlas Signal Connector for Signal C Upper Molex Picoblade 1 - Yellow 2 - Green 3 - Red 4 - Common"
- note added: "Atlas Signal Connector for Signal D Lower Molex Picoblade 1 - Yellow 2 - Green 3 - Red 4 - Common"
- note added: "Atlas Signal Connector for Signal D Upper Molex Picoblade 1 - Yellow 2 - Green 3 - Red 4 - Common"
- note added: "Signal A/B Common Terminal"
- note added: "Signal B-Lower - Green LED"
- note added: "Signal B-Lower - Red LED"
- note added: "Signal B-Lower - Yellow LED"
- note added: "Signal B-Upper - Green LED"
- note added: "Signal B-Upper - Red LED"
- note added: "Signal B-Upper - Yellow LED"
- note added: "Signal C-Lower - Green LED"
- note added: "Signal C-Lower - Red LED"
- note added: "Signal C-Lower - Yellow LED"
- note added: "Signal C-Upper - Green LED"
- note added: "Signal C-Upper - Red LED"
- note added: "Signal C-Upper - Yellow LED"
- note added: "Signal C/D Common Terminal"
- note added: "Signal D-Lower - Green LED"
- note added: "Signal D-Lower - Red LED"
- note added: "Signal D-Lower - Yellow LED"
- note added: "Signal D-Upper - Green LED"
- note added: "Signal D-Upper - Red LED"
- note added: "Signal D-Upper - Yellow LED"
- note removed: "7-Bit I2C Addr = 0x40"
- note removed: "7-Bit I2C Addr = 0x41"
- note removed: "Atlas Signal Connector for Signal A-Lower Molex Picoblade 1 - Yellow 2 - Green 3 - Red 4 - Common"
- note removed: "Signals Common Terminal"
- moved on the sheet: C35, J32, J33, J34, J35, J36, J37, J38, J39
