File: kicad/mss-xcade/mss-xcade.kicad_sch (KiCad schematic)
At the start: 128 parts

Commit message: More updates
Parts:
- removed JP? (x2): Conn_01x02, Connector_PinHeader_2.54mm:PinHeader_1x02_P2.54mm_Vertical, symbol Connector_Generic:Conn_01x02
- added D?: WS2812B, LED_SMD:LED_WS2812B_PLCC4_5.0x5.0mm_P3.2mm, symbol LED:WS2812B
- added SW?: FSM4JSMATR, ISE_Generic:TE_FSM4JSMA, symbol dk_Tactile-Switches:FSM4JSMATR
- added SW? (x2): SW_DIP_x08, symbol Switch:SW_DIP_x08
Connections:
- net +5V: now also D?.1 (VDD)
- net GND: now also D?.3 (VSS), SW?.3, SW?.4
- net ~{RST}: now also SW?.1, SW?.2
- net at U?.26 (GPIO45): now also D?.4 (DIN)
Other:
- note added: "TO DO: - irsense and bd1 inputs - config switches and how to use them - status led and reset stuff on esp32"
- moved on the sheet: C?

Commit message: More updates
Parts:
- removed J?: SM04B-SRSS, Connector_JST:JST_SH_SM04B-SRSS-TB_1x04-1MP_P1.00mm_Horizontal, symbol Connector_Generic_MountingPin:Conn_01x04_MountingPin
- added C? (x2): 0.1uF, Capacitor_SMD:C_0805_2012Metric, symbol Device:C
- added D? (x2): AMBER, LED_SMD:LED_0805_2012Metric, symbol Device:LED
- added J? (x13): SM04B-SRSS, Connector_JST:JST_SH_SM04B-SRSS-TB_1x04-1MP_P1.00mm_Horizontal, symbol Connector_Generic_MountingPin:Conn_01x04_MountingPin
- added J?: Screw_Terminal_01x08, symbol Connector:Screw_Terminal_01x08
- added R? (x2): 10k, Resistor_SMD:R_0805_2012Metric, symbol Device:R_US
- added R? (x2): 1k, Resistor_SMD:R_0805_2012Metric, symbol Device:R_US
- added U?: PCA9555D, Package_SO:SOIC-24W_7.5x15.4mm_P1.27mm, symbol Interface_Expansion:PCA9555D
- added U?: PCA9548APW, Package_SO:TSSOP-24_4.4x7.8mm_P0.65mm, symbol Interface_Expansion:PCA9548APW
Connections:
- net +3.3V: now also R?.2, C?.1, J?.2 (Pin_2), J?.2 (Pin_2), J?.2 (Pin_2), R?.2, R?.2, U?.24 (VCC)
- net +5V: now also C?.1, J?.1 (Pin_1), J?.2 (Pin_2), J?.2 (Pin_2), J?.2 (Pin_2), J?.2 (Pin_2), J?.2 (Pin_2), J?.2 (Pin_2), R?.2, R?.2, U?.2 (A1), U?.24 (VDD)
- net BOOT: now also SW?.1
- net GND: now also SW?.10, SW?.10, SW?.11, SW?.11, SW?.12, SW?.12, SW?.13, SW?.13, SW?.14, SW?.14, SW?.15, SW?.15, SW?.16, SW?.16, SW?.9, SW?.9, C?.2, C?.2, J?.1 (Pin_1), J?.1 (Pin_1), J?.1 (Pin_1), J?.1 (Pin_1), J?.1 (Pin_1), J?.1 (Pin_1), J?.1 (Pin_1), J?.1 (Pin_1), J?.1 (Pin_1), J?.1 (Pin_1), J?.1 (Pin_1), J?.1 (Pin_1), J?.1 (Pin_1), J?.8 (Pin_8), J?.MP (MountPin), J?.MP (MountPin), J?.MP (MountPin), J?.MP (MountPin), J?.MP (MountPin), J?.MP (MountPin), J?.MP (MountPin), J?.MP (MountPin), J?.MP (MountPin), J?.MP (MountPin), J?.MP (MountPin), J?.MP (MountPin), J?.MP (MountPin), U?.1 (A0), U?.12 (GND), U?.12 (VSS), U?.2 (A1), U?.21 (A0), U?.21 (A2), U?.3 (A2)
- net SCL: now also U?.22 (SCL), U?.5 (SC0)
- net SDA: now also U?.23 (SDA), U?.4 (SD0)
- net CONF_SW9: now reaches U?.12 (GPIO8)
- net CONF_SW9: now also SW?.1
- net CONF_SW4: now reaches U?.15 (GPIO3)
- net CONF_SW4: now also SW?.4
- net CONF_SW10: now reaches U?.17 (GPIO9)
- net CONF_SW10: now also SW?.2
- net CONF_SW11: now reaches U?.18 (GPIO10)
- net CONF_SW11: now also SW?.3
- net CONF_SW12: now reaches U?.19 (GPIO11)
- net CONF_SW12: now also SW?.4
- net CONF_SW13: now reaches U?.20 (GPIO12)
- net CONF_SW13: now also SW?.5
- net CONF_SW14: now reaches U?.21 (GPIO13)
- net CONF_SW14: now also SW?.6
- net CONF_SW15: now reaches U?.22 (GPIO14)
- net CONF_SW15: now also SW?.7
- net at Q?.2 (S), U?.24 (GPIO33): now also R?.1, U?.23 (SDA)
- net at Q?.2 (S), U?.25 (GPIO34): now also R?.1, U?.22 (SCL)
- net at U?.28 (GPIO35): now also U?.3 (~{RESET})
- net CONF_SW16: now reaches U?.29 (GPIO36)
- net CONF_SW16: now also SW?.8
- net CONF_SW3: now reaches U?.38 (GPIO2)
- net CONF_SW3: now also SW?.3
- net CONF_SW2: now reaches U?.39 (GPIO1)
- net CONF_SW2: now also SW?.2
- net CONF_SW5: now reaches U?.4 (GPIO4)
- net CONF_SW5: now also SW?.5
- net CONF_SW6: now reaches U?.5 (GPIO5)
- net CONF_SW6: now also SW?.6
- net CONF_SW7: now reaches U?.6 (GPIO6)
- net CONF_SW7: now also SW?.7
- net CONF_SW8: now reaches U?.7 (GPIO7)
- net CONF_SW8: now also SW?.8
- net at U?.22 (LED15): now also D?.1 (K) (x2)
- new net: D?.2 (A), R?.1 (x2)
- new net SCL_EXP_1: J?.4 (Pin_4), U?.7 (SC1)
- new net SCL_EXP_2: J?.4 (Pin_4), U?.9 (SC2)
- new net SCL_EXP_3: J?.4 (Pin_4), U?.11 (SC3)
- new net SCL_EXP_4: U?.14 (SC4)
- new net SCL_EXP_5: U?.16 (SC5)
- new net SCL_EXP_6: U?.18 (SC6)
- new net SCL_EXP_7: U?.20 (SC7)
- new net SDA_EXP_1: J?.3 (Pin_3), U?.6 (SD1)
- new net SDA_EXP_2: J?.3 (Pin_3), U?.8 (SD2)
- new net SDA_EXP_3: J?.3 (Pin_3), U?.10 (SD3)
- new net SDA_EXP_4: U?.13 (SD4)
- new net SDA_EXP_5: U?.15 (SD5)
- new net SDA_EXP_6: U?.17 (SD6)
- new net SDA_EXP_7: U?.19 (SD7)
- new net SENSOR_IN_0: J?.3 (Pin_3), U?.4 (IO0_0)
- new net SENSOR_IN_1: J?.3 (Pin_3), U?.5 (IO0_1)
- new net SENSOR_IN_10: J?.2 (Pin_2), U?.15 (IO1_2)
- new net SENSOR_IN_11: J?.3 (Pin_3), U?.16 (IO1_3)
- new net SENSOR_IN_12: J?.4 (Pin_4), U?.17 (IO1_4)
- new net SENSOR_IN_13: J?.5 (Pin_5), U?.18 (IO1_5)
- new net SENSOR_IN_14: J?.6 (Pin_6), U?.19 (IO1_6)
- new net SENSOR_IN_15: J?.7 (Pin_7), U?.20 (IO1_7)
- new net SENSOR_IN_2: J?.3 (Pin_3), U?.6 (IO0_2)
- new net SENSOR_IN_3: J?.3 (Pin_3), U?.7 (IO0_3)
- new net SENSOR_IN_4: J?.3 (Pin_3), U?.8 (IO0_4)
- new net SENSOR_IN_5: J?.3 (Pin_3), U?.9 (IO0_5)
- new net SENSOR_IN_6: J?.3 (Pin_3), U?.10 (IO0_6)
- new net SENSOR_IN_7: J?.3 (Pin_3), U?.11 (IO0_7)
- new net SENSOR_IN_8: J?.3 (Pin_3), U?.13 (IO1_0)
- new net SENSOR_IN_9: J?.3 (Pin_3), U?.14 (IO1_1)
Other:
- sheet MSS Interface renamed MSS Bus Interface
- note added: "7-Bit I2C Addr = 0x22"
- note added: "7-Bit I2C Addr = 0x40"
- note added: "7-Bit I2C Addr = 0x41"
- note added: "7-Bit I2C Addr = 0x70"
- note added: "Note: Either install level- shifting transistors or PCA9548, not both"
- note removed: "IRSense"
- note removed: "Isolated 4-Channel MSS Bus Interface Schematic Sheet"
- note removed: "TO DO: - irsense and bd1 inputs - config switches and how to use them - status led and reset stuff on esp32"
- moved on the sheet: D?, H1, H2, H3, H4, SW?, U?

Commit message: xcade upates
Parts:
- gave numbers to parts that had none: 149

Commit message: Refactor signal drivers to their own schematic and add picoblade connectors
Parts:
- removed C10, C2: 1uF, Capacitor_SMD:C_0805_2012Metric, symbol Device:C
- removed C13: 0.1uF, Capacitor_SMD:C_0805_2012Metric, symbol Device:C
- removed D10, D7: AMBER, LED_SMD:LED_0805_2012Metric, symbol Device:LED
- removed J10, J12, J13, J14, J2, J3, J4, J5, J6, J7, J8, J9: Screw_Terminal_01x02, TerminalBlock_MetzConnect:TerminalBlock_MetzConnect_Type059_RT06303HBWC_1x03_P3.50mm_Horizontal, symbol Connector:Screw_Terminal_01x03
- removed J17, J18, J19, J20, J21, J22, J23, J24, J26, J27: SM04B-SRSS, Connector_JST:JST_SH_SM04B-SRSS-TB_1x04-1MP_P1.00mm_Horizontal, symbol Connector_Generic_MountingPin:Conn_01x04_MountingPin
- removed J28: Screw_Terminal_01x08, symbol Connector:Screw_Terminal_01x08
- removed JP1, JP10, JP11, JP12, JP13, JP14, JP15, JP16, JP17, JP18, JP19, JP2, JP20, JP21, JP22, JP23, JP24, JP3, JP4, JP5, JP6, JP7, JP8, JP9: SolderJumper_2_Open, Jumper:SolderJumper-2_P1.3mm_Open_RoundedPad1.0x1.5mm, symbol Jumper:SolderJumper_2_Open
- removed Q1, Q2: BSS138, Package_TO_SOT_SMD:SOT-23, symbol Transistor_FET:BSS138
- removed R1, R11, R14, R19, R20, R22, R23, R24, R25, R26, R27, R28, R29, R30, R31, R32, R33, R35, R4, R5, R6, R7, R8, R9: 330, Resistor_SMD:R_0805_2012Metric, symbol Device:R_US
- removed R12, R13, R15, R16, R21, R34: 1k, Resistor_SMD:R_0805_2012Metric, symbol Device:R_US
- removed TP1, TP10, TP11, TP12, TP13, TP14, TP15, TP16, TP17, TP18, TP19, TP20, TP21, TP22, TP23, TP24, TP25, TP26, TP4, TP5, TP6, TP7, TP8, TP9: TestPoint, TestPoint:TestPoint_Pad_D2.0mm, symbol Connector:TestPoint
- removed U3, U6: PCA9635, Package_SO:TSSOP-28_4.4x9.7mm_P0.65mm, symbol Driver_LED:PCA9635
- removed U7: PCA9555D, Package_SO:SOIC-24W_7.5x15.4mm_P1.27mm, symbol Interface_Expansion:PCA9555D
- added J?: BM06B-SRSS, Connector_JST:JST_SH_BM06B-SRSS-TB_1x06-1MP_P1.00mm_Vertical, symbol Connector_Generic_MountingPin:Conn_01x06_MountingPin
- added J?: SM04B-SRSS, Connector_JST:JST_SH_SM04B-SRSS-TB_1x04-1MP_P1.00mm_Horizontal, symbol Connector_Generic_MountingPin:Conn_01x04_MountingPin
- added R? (x4): 1k, Resistor_SMD:R_0805_2012Metric, symbol Device:R_US
Connections:
- net +3.3V: now also J?.5 (Pin_5); no longer J15.2 (Pin_2), J16.2 (Pin_2), J25.2 (Pin_2)
- net +5V: now also J15.2 (Pin_2), J16.2 (Pin_2), J25.2 (Pin_2), J?.2 (Pin_2), R?.2, R?.2
- net GND: now also J?.1 (Pin_1), J?.2 (Pin_2), J?.6 (Pin_6), J?.MP (MountPin), J?.MP (MountPin)
- net SCL: now also J?.4 (Pin_4), R?.1
- net SDA: now also J?.3 (Pin_3), R?.1
- net VPWR: now also J?.1 (Pin_1)
- net CAN_H: now reaches U4.32 (GPIO39)
- net CAN_H: now also J?.3 (Pin_3)
- net CAN_L: now reaches U4.33 (GPIO40)
- net CAN_L: now also J?.4 (Pin_4)
- net EN4: no longer names the net of U4.23 (GPIO21)
- net SCL_EXP_1: no longer names the net of J15.4 (Pin_4), U5.7 (SC1)
- net SCL_EXP_2: no longer names the net of J16.4 (Pin_4), U5.9 (SC2)
- net SCL_EXP_3: no longer names the net of J25.4 (Pin_4), U5.11 (SC3)
- net SDA_EXP_1: no longer names the net of J15.3 (Pin_3), U5.6 (SD1)
- net SDA_EXP_2: no longer names the net of J16.3 (Pin_3), U5.8 (SD2)
- net SDA_EXP_3: no longer names the net of J25.3 (Pin_3), U5.10 (SD3)
- new net: R?.1, R?.2 (x2)
Other:
- added sheet Signals & Sensors (mss-xcade-signal-drivers.kicad_sch)
- note added: "Expansion Port 2"
- note added: "Expansion Port 3"
- note added: "Expansion Port 4"
- note added: "Input Jack for Secondary Boards DNI on primary"
- note added: "LCC Expansion Connector"
- note removed: "7-Bit I2C Addr = 0x22"
- note removed: "7-Bit I2C Addr = 0x40"
- note removed: "7-Bit I2C Addr = 0x41"
- note removed: "Note: Either install level- shifting transistors or PCA9548, not both"
- note removed: "Signal A1 - Common Anode"
- note removed: "Signal A1 - Green LED Cathode"
- note removed: "Signal A1 - Red LED Cathode"
- note removed: "Signal A1 - Yellow LED Cathode"
- note removed: "Signal A2 - Common Anode"
- note removed: "Signal A2 - Green LED Cathode"
- note removed: "Signal A2 - Red LED Cathode"
- note removed: "Signal A2 - Yellow LED Cathode"
- note removed: "Signal B1 - Common Anode"
- note removed: "Signal B1 - Green LED Cathode"
- note removed: "Signal B1 - Red LED Cathode"
- note removed: "Signal B1 - Yellow LED Cathode"
- note removed: "Signal B2 - Common Anode"
- note removed: "Signal B2 - Green LED Cathode"
- note removed: "Signal B2 - Red LED Cathode"
- note removed: "Signal B2 - Yellow LED Cathode"
- note removed: "Signal C1 - Common Anode"
- note removed: "Signal C1 - Green LED Cathode"
- note removed: "Signal C1 - Red LED Cathode"
- note removed: "Signal C1 - Yellow LED Cathode"
- note removed: "Signal C2 - Common Anode"
- note removed: "Signal C2 - Green LED Cathode"
- note removed: "Signal C2 - Red LED Cathode"
- note removed: "Signal C2 - Yellow LED Cathode"
- note removed: "Signal D1 - Common Anode"
- note removed: "Signal D1 - Green LED Cathode"
- note removed: "Signal D1 - Red LED Cathode"
- note removed: "Signal D1 - Yellow LED Cathode"
- note removed: "Signal D2 - Common Anode"
- note removed: "Signal D2 - Green LED Cathode"
- note removed: "Signal D2 - Red LED Cathode"
- note removed: "Signal D2 - Yellow LED Cathode"
- title: MSS Cascade Basic v1.0 -> MSS Cascade Advanced
- moved on the sheet: C1, C11, C12, C3, C4, C5, C6, C7, C8, C9, D1, D2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

Commit message: First cut of xcade PCB
Parts:
- removed C12: 10uF, Capacitor_SMD:C_0805_2012Metric, symbol Device:C
- removed J11: 690-005-299-043, digikey-footprints:USB_Mini_B_Female_690-005-299-043, symbol dk_USB-DVI-HDMI-Connectors:690-005-299-043
- removed J?: BM06B-SRSS, Connector_JST:JST_SH_BM06B-SRSS-TB_1x06-1MP_P1.00mm_Vertical, symbol Connector_Generic_MountingPin:Conn_01x06_MountingPin
- removed J?: SM04B-SRSS, Connector_JST:JST_SH_SM04B-SRSS-TB_1x04-1MP_P1.00mm_Horizontal, symbol Connector_Generic_MountingPin:Conn_01x04_MountingPin
- removed SW3: SW_DIP_x08, symbol Switch:SW_DIP_x08
- removed U5: PCA9548APW, Package_SO:TSSOP-24_4.4x7.8mm_P0.65mm, symbol Interface_Expansion:PCA9548APW
- added H5, H6: MountingHole, MountingHole:MountingHole_3.2mm_M3_ISO14580_Pad, symbol Mechanical:MountingHole_Pad
- added J3: 690-005-299-043, ISE_UltraLibrarian:EDAC_690-005-299-043, symbol ISE_UltraLibrarian:690-005-299-043
- added J5: Conn_02x03_Odd_Even, Connector_PinHeader_2.54mm:PinHeader_2x03_P2.54mm_Vertical, symbol Connector_Generic:Conn_02x03_Odd_Even
- added R10, R11: 0, Resistor_SMD:R_0805_2012Metric, symbol Device:R_US
- added REF1, REF2, REF3: Fiducial, symbol Mechanical:Fiducial
- added U3: PCA9546ADR, Package_SO:SOIC-16_3.9x9.9mm_P1.27mm, symbol ISE_Generic:PCA9546ADR
- SW2: footprint (none) -> Button_Switch_SMD:SW_DIP_SPSTx08_Slide_6.7x21.88mm_W8.61mm_P2.54mm_LowProfile
- U1: footprint (none) -> Package_TO_SOT_SMD:SOT-223-3_TabPin2
- U4: footprint Espressif:ESP32-S2-SOLO -> ISE_Generic:ESP32-S2-SOLO
- gave numbers to parts that had none: 4
- renumbered C3 to C2, C4 to C3, C5 to C4, C6 to C5, C7 to C6, C9 to C7, C11 to C9, D8 to D7, D9 to D8, J15 to J2, J16 to J4, J25 to J6, R2 to R1, R3 to R2, R10 to R7, R17 to R8, R18 to R9, TP2 to TP1, TP3 to TP2
Connections:
- net CONF_SW10 is gone; now on net CONF_SW8: U4.17 (GPIO9)
- net CONF_SW11 is gone; now on net CONF_SW7: U4.18 (GPIO10)
- net CONF_SW12 is gone; now on net CONF_SW6: U4.19 (GPIO11)
- net CONF_SW13 is gone; now on net CONF_SW5: U4.20 (GPIO12)
- net CONF_SW14 is gone; now on net CONF_SW4: U4.21 (GPIO13)
- net CONF_SW15 is gone; now on net CONF_SW3: U4.22 (GPIO14)
- net CONF_SW16 is gone; now on an unnamed net: U4.29 (GPIO36)
- net +3.3V: now also J5.6 (Pin_6), U3.16 (VCC)
- net +5V: now also J2.MP (MountPin), J4.MP (MountPin), J6.MP (MountPin)
- net BOOT: now also SW2.9; no longer SW2.1
- net CONF_SW2: now also SW2.10, U4.23 (GPIO21); no longer SW2.2, U4.39 (GPIO1)
- net CONF_SW3: now also SW2.11; no longer SW2.3, U4.38 (GPIO2)
- net CONF_SW4: now also SW2.12; no longer SW2.4, U4.15 (GPIO3)
- net CONF_SW5: now also SW2.13; no longer SW2.5, U4.4 (GPIO4)
- net CONF_SW6: now also SW2.14; no longer SW2.6, U4.5 (GPIO5)
- net CONF_SW7: now also SW2.15; no longer SW2.7, U4.6 (GPIO6)
- net CONF_SW8: now also SW2.16; no longer SW2.8, U4.7 (GPIO7)
- net D+: now also J3.3 (D+)
- net D-: now also J3.2 (D-)
- net GND: now also SW2.1, SW2.2, SW2.3, SW2.4, SW2.5, SW2.6, SW2.7, SW2.8, J3.5 (GND), J3.S1 (SHIELD), J5.2 (Pin_2), U3.1 (A0), U3.13 (A2), U3.2 (A1), U3.8 (GND); no longer J2.MP (MountPin), J4.MP (MountPin), J6.MP (MountPin), SW2.10, SW2.11, SW2.12, SW2.13, SW2.14, SW2.15, SW2.16, SW2.9
- net SCL: now also R10.2, U3.5 (SCL0)
- net SDA: now also R11.2, U3.4 (SDA0)
- net at J6.3 (Pin_3): now also U3.11 (SDA3)
- net at J6.4 (Pin_4): now also U3.12 (SCL3)
- net at R8.1: now also U3.15 (SDA); no longer U4.24 (GPIO33)
- net at U4.25 (GPIO34): no longer R9.1
- net at U4.28 (GPIO35): now also U3.3 (~{RESET})
- net at U4.30 (GPIO37): now also R9.1, U3.14 (SCL)
- net CAN_AUX1: now reaches U4.34 (GPIO41)
- net CAN_AUX1: now also J5.1 (Pin_1)
- net CAN_AUX2: now reaches U4.35 (GPIO42)
- net CAN_AUX2: now also J5.5 (Pin_5)
- net at D7.2 (A): now also J3.1 (VCC)
- net at J4.3 (Pin_3): now also U3.9 (SDA2)
- net at J4.4 (Pin_4): now also U3.10 (SCL2)
- net at J2.3 (Pin_3): now also R11.1, U3.6 (SDA1)
- net at J2.4 (Pin_4): now also R10.1, U3.7 (SCL1)
- net CAN_H renamed CAN_TX
- net CAN_TX: now also J5.3 (Pin_3)
- net CAN_L renamed CAN_RX
- net CAN_RX: now also J5.4 (Pin_4)
- net CONF_SW9: no longer names the net of U4.12 (GPIO8)
Other:
- note added: "DNI on master Install on expansion units"
- note removed: "Input Jack for Secondary Boards DNI on primary"
- moved on the sheet: C9, H1, H2, H3, H4, SW2
